File: ModularSeries/DualAttenuverter/DualAttenuverter.brd (EAGLE design)
At the start: 48 x 47 mm, 33 parts, among them IC1 TL0X4_DIP, IC2 LM358_DIP

Commit message: Library updated, variants consolidated
Parts:
- IC1: value TL0X4_DIP -> (none)
- IC2: value LM358_DIP -> LM358
Changed lines of the file:
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@@
 <attribute name="VALUE" x="45.339" y="17.534" size="1.27" layer="27" ratio="10" rot="R180"/>
 </element>
-<element name="IC1" library="ElectricNoodleBox" package="DIL14" package3d_urn="urn:adsk.eagle:package:16407/2" value="TL0X4_DIP" x="19.05" y="23.63" smashed="yes" rot="R180">
+<element name="IC1" library="ElectricNoodleBox" package="DIL14" package3d_urn="urn:adsk.eagle:package:16407/2" value="" x="19.05" y="23.63" smashed="yes" rot="R180">
 <attribute name="NAME" x="28.321" y="27.948" size="1.27" layer="25" ratio="10" rot="R270"/>
 <attribute name="VALUE" x="25.781" y="24.265" size="1.27" layer="27" ratio="10" rot="R180"/>
@@
 <attribute name="VALUE" x="17.145" y="46.998" size="0.6096" layer="27" font="vector" ratio="20"/>
 </element>
-<element name="IC2" library="ElectricNoodleBox" package="DIL08" package3d_urn="urn:adsk.eagle:package:29519/2" value="LM358_DIP" x="41.91" y="23.63" smashed="yes" rot="R270">
+<element name="IC2" library="ElectricNoodleBox" package="DIL08" package3d_urn="urn:adsk.eagle:package:29519/2" value="LM358" x="41.91" y="23.63" smashed="yes" rot="R270">
 <attribute name="NAME" x="38.989" y="28.964" size="1.27" layer="25" ratio="10"/>
 <attribute name="VALUE" x="41.275" y="27.186" size="1.27" layer="27" ratio="10" rot="R270"/>
