File: ModularSeries/DCModuleSplitSupply/DCModuleSplitSupply.sch (EAGLE design)
At the start: 26 parts, among them J1 2XMOLEX, J2 4XMOLEX, J3 4XMOLEX, J4 4XMOLEX, J5 4XMOLEX, J6 2XMOLEX, J7 2XMOLEX, J8 4XMOLEX

Commit message: Library updated, variants consolidated
Parts:
- PREF1, PREF2: device ElectricNoodleBox:LM4040_TO92 -> ElectricNoodleBox:LM4040TH
Connections:
- net +10VREF: now also PREF1.CATHODE; no longer PREF1.V+
- net -10VREF: now also PREF2.ANODE; no longer PREF2.V-
- net AGND: now also PREF1.ANODE, PREF2.CATHODE; no longer PREF1.V-, PREF2.V+
Changed lines of the file:
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@@
 <part name="C2" library="rcl" library_urn="urn:adsk.eagle:library:334" deviceset="CPOL-EU" device="E2-5" package3d_urn="urn:adsk.eagle:package:23346/2" value="10µF"/>
 <part name="C3" library="rcl" library_urn="urn:adsk.eagle:library:334" deviceset="CPOL-EU" device="E2-5" package3d_urn="urn:adsk.eagle:package:23346/2" value="10µF"/>
-<part name="PREF1" library="ElectricNoodleBox" deviceset="LM4040_TO92" device="" value="LM4040 10V"/>
-<part name="PREF2" library="ElectricNoodleBox" deviceset="LM4040_TO92" device="" value="LM4040 10V"/>
+<part name="PREF1" library="ElectricNoodleBox" deviceset="LM4040" device="TH" value="LM4040 10V"/>
+<part name="PREF2" library="ElectricNoodleBox" deviceset="LM4040" device="TH" value="LM4040 10V"/>
 <part name="P+1" library="supply1" library_urn="urn:adsk.eagle:library:371" deviceset="+12V" device=""/>
 <part name="P-1" library="supply1" library_urn="urn:adsk.eagle:library:371" deviceset="-12V" device=""/>
@@
 <pinref part="R1" gate="G$1" pin="2"/>
 <wire x1="99.06" y1="55.88" x2="104.14" y2="55.88" width="0.1524" layer="91"/>
-<pinref part="PREF1" gate="G$1" pin="V+"/>
+<pinref part="PREF1" gate="G$1" pin="CATHODE"/>
 <wire x1="104.14" y1="55.88" x2="104.14" y2="53.34" width="0.1524" layer="91"/>
 <wire x1="104.14" y1="55.88" x2="104.14" y2="58.42" width="0.1524" layer="91"/>
@@
 <pinref part="R2" gate="G$1" pin="2"/>
 <wire x1="99.06" y1="25.4" x2="104.14" y2="25.4" width="0.1524" layer="91"/>
-<pinref part="PREF2" gate="G$1" pin="V-"/>
+<pinref part="PREF2" gate="G$1" pin="ANODE"/>
 <wire x1="104.14" y1="25.4" x2="104.14" y2="27.94" width="0.1524" layer="91"/>
 <wire x1="104.14" y1="25.4" x2="104.14" y2="22.86" width="0.1524" layer="91"/>
@@
 <junction x="83.82" y="40.64"/>
 <wire x1="83.82" y1="40.64" x2="104.14" y2="40.64" width="0.1524" layer="91"/>
-<pinref part="PREF1" gate="G$1" pin="V-"/>
+<pinref part="PREF1" gate="G$1" pin="ANODE"/>
 <wire x1="104.14" y1="40.64" x2="104.14" y2="43.18" width="0.1524" layer="91"/>
-<pinref part="PREF2" gate="G$1" pin="V+"/>
+<pinref part="PREF2" gate="G$1" pin="CATHODE"/>
 <wire x1="104.14" y1="40.64" x2="104.14" y2="38.1" width="0.1524" layer="91"/>
 <junction x="104.14" y="40.64"/>

Commit message: DC Split Supply layout revision
Parts:
- added P6: 4XMOLEX, ElectricNoodleBox:4XMOLEX
- renumbered J1 to VIN, J2 to P1, J3 to P2, J4 to P3, J5 to P4, J6 to VREF1, J7 to VREF2, J8 to P5
Connections:
- net +12V: now also P6.1
- net -12V: now also P6.4
- net AGND: now also P6.2, P6.3
