File: ModularSeries/PortalsDualExpVCA/PortalsDualExpVCA.brd (EAGLE design)
At the start: 47 x 95 mm, 71 parts, among them Q1 2N3906, Q2 2N3906, Q3 2N3906, Q4 2N3906

Commit message: Updates to Portals and Knives, Panel layout for Prism and Knives added
Parts:
- R1, R18, R35, R36: value 22K -> 15K
- R14, R31: value 100Ω -> 47Ω
- R17, R26, R34, R9: value 75K -> 47K
- R22, R5: value 33K -> 22K
Changed lines of the file:
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@@
 <attribute name="VALUE" x="42.545" y="64" size="1.27" layer="27" ratio="10"/>
 </element>
-<element name="R1" library="rcl" library_urn="urn:adsk.eagle:library:334" package="0207/10" package3d_urn="urn:adsk.eagle:package:23491/2" value="22K" x="11.43" y="32.25" smashed="yes">
+<element name="R1" library="rcl" library_urn="urn:adsk.eagle:library:334" package="0207/10" package3d_urn="urn:adsk.eagle:package:23491/2" value="15K" x="11.43" y="32.25" smashed="yes">
 <attribute name="NAME" x="9.652" y="31.234" size="1.27" layer="25" ratio="10"/>
 <attribute name="POPULARITY" value="81" x="82.55" y="1.77" size="1.778" layer="27" display="off"/>
@@
 <attribute name="VALUE" x="34.87" y="10.52" size="1.27" layer="27"/>
 </element>
-<element name="R14" library="rcl" library_urn="urn:adsk.eagle:library:334" package="0207/10" package3d_urn="urn:adsk.eagle:package:23491/2" value="100Ω" x="39.37" y="10.66" smashed="yes">
+<element name="R14" library="rcl" library_urn="urn:adsk.eagle:library:334" package="0207/10" package3d_urn="urn:adsk.eagle:package:23491/2" value="47Ω" x="39.37" y="10.66" smashed="yes">
 <attribute name="NAME" x="37.592" y="9.644" size="1.27" layer="25" ratio="10"/>
 <attribute name="POPULARITY" value="81" x="71.12" y="-37.6" size="1.778" layer="27" display="off"/>
@@
 <attribute name="VALUE" x="41.6306" y="40.505" size="1.27" layer="27" ratio="10" rot="R180"/>
 </element>
-<element name="R17" library="rcl" library_urn="urn:adsk.eagle:library:334" package="0207/10" package3d_urn="urn:adsk.eagle:package:23491/2" value="75K" x="11.43" y="19.55" smashed="yes">
+<element name="R17" library="rcl" library_urn="urn:adsk.eagle:library:334" package="0207/10" package3d_urn="urn:adsk.eagle:package:23491/2" value="47K" x="11.43" y="19.55" smashed="yes">
 <attribute name="NAME" x="9.652" y="18.534" size="1.27" layer="25" ratio="10"/>
 <attribute name="POPULARITY" value="81" x="81.28" y="-28.71" size="1.778" layer="27" display="off"/>
@@
 <attribute name="VALUE" x="9.1694" y="18.915" size="1.27" layer="27" ratio="10"/>
 </element>
-<element name="R18" library="rcl" library_urn="urn:adsk.eagle:library:334" package="0207/10" package3d_urn="urn:adsk.eagle:package:23491/2" value="22K" x="11.43" y="62.73" smashed="yes">
+<element name="R18" library="rcl" library_urn="urn:adsk.eagle:library:334" package="0207/10" package3d_urn="urn:adsk.eagle:package:23491/2" value="15K" x="11.43" y="62.73" smashed="yes">
 <attribute name="NAME" x="9.652" y="61.714" size="1.27" layer="25" ratio="10"/>
 <attribute name="POPULARITY" value="81" x="30.48" y="9.39" size="1.778" layer="27" display="off"/>
@@
 <attribute name="VALUE" x="27.6606" y="60.825" size="1.27" layer="27" ratio="10" rot="R180"/>
 </element>
-<element name="R22" library="rcl" library_urn="urn:adsk.eagle:library:334" package="0207/10" package3d_urn="urn:adsk.eagle:package:23491/2" value="33K" x="25.4" y="57.65" smashed="yes" rot="R180">
+<element name="R22" library="rcl" library_urn="urn:adsk.eagle:library:334" package="0207/10" package3d_urn="urn:adsk.eagle:package:23491/2" value="22K" x="25.4" y="57.65" smashed="yes" rot="R180">
 <attribute name="NAME" x="23.622" y="56.904" size="1.27" layer="25" ratio="10"/>
 <attribute name="POPULARITY" value="81" x="-44.45" y="110.99" size="1.778" layer="27" rot="R180" display="off"/>
@@
 <attribute name="VALUE" x="9.1694" y="79.875" size="1.27" layer="27" ratio="10"/>
 </element>
-<element name="R26" library="rcl" library_urn="urn:adsk.eagle:library:334" package="0207/10" package3d_urn="urn:adsk.eagle:package:23491/2" value="75K" x="11.43" y="77.97" smashed="yes">
+<element name="R26" library="rcl" library_urn="urn:adsk.eagle:library:334" package="0207/10" package3d_urn="urn:adsk.eagle:package:23491/2" value="47K" x="11.43" y="77.97" smashed="yes">
 <attribute name="NAME" x="9.652" y="76.954" size="1.27" layer="25" ratio="10"/>
 <attribute name="POPULARITY" value="81" x="68.58" y="19.55" size="1.778" layer="27" display="off"/>
@@
 <attribute name="VALUE" x="34.87" y="76.56" size="1.27" layer="27"/>
 </element>
-<element name="R31" library="rcl" library_urn="urn:adsk.eagle:library:334" package="0207/10" package3d_urn="urn:adsk.eagle:package:23491/2" value="100Ω" x="39.37" y="84.32" smashed="yes">
+<element name="R31" library="rcl" library_urn="urn:adsk.eagle:library:334" package="0207/10" package3d_urn="urn:adsk.eagle:package:23491/2" value="47Ω" x="39.37" y="84.32" smashed="yes">
 <attribute name="NAME" x="37.592" y="83.304" size="1.27" layer="25" ratio="10"/>
 <attribute name="POPULARITY" value="81" x="83.82" y="20.82" size="1.778" layer="27" display="off"/>
@@
 <attribute name="VALUE" x="37.1094" y="54.475" size="1.27" layer="27" ratio="10"/>
 </element>
-<element name="R34" library="rcl" library_urn="urn:adsk.eagle:library:334" package="0207/10" package3d_urn="urn:adsk.eagle:package:23491/2" value="75K" x="11.43" y="75.43" smashed="yes">
+<element name="R34" library="rcl" library_urn="urn:adsk.eagle:library:334" package="0207/10" package3d_urn="urn:adsk.eagle:package:23491/2" value="47K" x="11.43" y="75.43" smashed="yes">
 <attribute name="NAME" x="9.652" y="74.414" size="1.27" layer="25" ratio="10"/>
 <attribute name="POPULARITY" value="81" x="30.48" y="6.85" size="1.778" layer="27" display="off"/>
@@
 <attribute name="VALUE" x="9.1694" y="74.795" size="1.27" layer="27" ratio="10"/>
 </element>
-<element name="R35" library="rcl" library_urn="urn:adsk.eagle:library:334" package="0207/10" package3d_urn="urn:adsk.eagle:package:23491/2" value="22K" x="11.43" y="34.79" smashed="yes">
+<element name="R35" library="rcl" library_urn="urn:adsk.eagle:library:334" package="0207/10" package3d_urn="urn:adsk.eagle:package:23491/2" value="15K" x="11.43" y="34.79" smashed="yes">
 <attribute name="NAME" x="9.652" y="33.774" size="1.27" layer="25" ratio="10"/>
 <attribute name="POPULARITY" value="81" x="43.18" y="-33.79" size="1.778" layer="27" display="off"/>
@@
 <attribute name="VALUE" x="9.1694" y="34.155" size="1.27" layer="27" ratio="10"/>
 </element>
-<element name="R36" library="rcl" library_urn="urn:adsk.eagle:library:334" package="0207/10" package3d_urn="urn:adsk.eagle:package:23491/2" value="22K" x="11.43" y="60.19" smashed="yes">
+<element name="R36" library="rcl" library_urn="urn:adsk.eagle:library:334" package="0207/10" package3d_urn="urn:adsk.eagle:package:23491/2" value="15K" x="11.43" y="60.19" smashed="yes">
 <attribute name="NAME" x="9.652" y="59.174" size="1.27" layer="25" ratio="10"/>
 <attribute name="POPULARITY" value="81" x="55.88" y="-8.39" size="1.778" layer="27" display="off"/>
@@
 <attribute name="VALUE" x="27.6606" y="35.425" size="1.27" layer="27" ratio="10" rot="R180"/>
 </element>
-<element name="R5" library="rcl" library_urn="urn:adsk.eagle:library:334" package="0207/10" package3d_urn="urn:adsk.eagle:package:23491/2" value="33K" x="25.4" y="37.33" smashed="yes" rot="R180">
+<element name="R5" library="rcl" library_urn="urn:adsk.eagle:library:334" package="0207/10" package3d_urn="urn:adsk.eagle:package:23491/2" value="22K" x="25.4" y="37.33" smashed="yes" rot="R180">
 <attribute name="NAME" x="23.622" y="36.584" size="1.27" layer="25" ratio="10"/>
 <attribute name="POPULARITY" value="81" x="-31.75" y="75.43" size="1.778" layer="27" rot="R180" display="off"/>
@@
 <attribute name="VALUE" x="9.1694" y="13.835" size="1.27" layer="27" ratio="10"/>
 </element>
-<element name="R9" library="rcl" library_urn="urn:adsk.eagle:library:334" package="0207/10" package3d_urn="urn:adsk.eagle:package:23491/2" value="75K" x="11.43" y="17.01" smashed="yes">
+<element name="R9" library="rcl" library_urn="urn:adsk.eagle:library:334" package="0207/10" package3d_urn="urn:adsk.eagle:package:23491/2" value="47K" x="11.43" y="17.01" smashed="yes">
 <attribute name="NAME" x="9.652" y="15.994" size="1.27" layer="25" ratio="10"/>
 <attribute name="POPULARITY" value="81" x="55.88" y="-26.17" size="1.778" layer="27" display="off"/>
