File: ModularSeries/KnivesDualLoopingARFG/Panel/KnivesPanel.brd (EAGLE design)
At the start: 50.5 x 128.5 mm, 16 parts

Commit message: Panel for TimeSeeds added. TLHP core PCB added
Parts:
- added E$17: (no value), ElectricNoodleBox:LOGO20X20
Changed lines of the file:
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@@
 <layer number="20" name="Dimension" color="24" fill="1" visible="yes" active="yes"/>
 <layer number="21" name="tPlace" color="7" fill="1" visible="yes" active="yes"/>
-<layer number="22" name="bPlace" color="7" fill="1" visible="no" active="yes"/>
-<layer number="23" name="tOrigins" color="15" fill="1" visible="no" active="yes"/>
-<layer number="24" name="bOrigins" color="15" fill="1" visible="no" active="yes"/>
+<layer number="22" name="bPlace" color="7" fill="1" visible="yes" active="yes"/>
+<layer number="23" name="tOrigins" color="15" fill="1" visible="yes" active="yes"/>
+<layer number="24" name="bOrigins" color="15" fill="1" visible="yes" active="yes"/>
 <layer number="25" name="tNames" color="7" fill="1" visible="no" active="yes"/>
 <layer number="26" name="bNames" color="7" fill="1" visible="no" active="yes"/>
@@
 <element name="E$15" library="ElectricNoodleBox" package="MCDTS_BUTTON_ROUND_CUTOUT" value="" x="16" y="57" smashed="yes"/>
 <element name="E$16" library="ElectricNoodleBox" package="MCDTS_BUTTON_ROUND_CUTOUT" value="" x="16" y="43" smashed="yes"/>
+<element name="E$17" library="ElectricNoodleBox" package="LOGO20X20" value="" x="49" y="93" smashed="yes" rot="MR0"/>
 </elements>
 <signals>
