File: ModularSeries/Ffrydiau/Ffrydiau_core.brd (EAGLE design)
At the start: 100 x 49 mm, 85 parts, among them Q1 2N3906, Q2 2N3904, Q3 2N3906, Q4 2N3904

Commit message: Ffrydiau BOMs added
Parts:
- R28, R30: value 2K -> 100K
Changed lines of the file:
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@@
 </element>
 <element name="IC1" library="ElectricNoodleBox" package="DIL14" package3d_urn="urn:adsk.eagle:package:16407/2" value="" x="87.63" y="25.4" smashed="yes" rot="R180">
+<attribute name="CATALOGUE" value="3005140" x="87.63" y="25.4" size="1.778" layer="27" rot="R180" display="off"/>
 <attribute name="NAME" x="96.901" y="28.448" size="1.27" layer="25" ratio="10" rot="R270"/>
+<attribute name="RETAILER" value="Farnell" x="87.63" y="25.4" size="1.778" layer="27" rot="R180" display="off"/>
 <attribute name="VALUE" x="94.361" y="26.035" size="1.27" layer="27" ratio="10" rot="R180"/>
 </element>
 <element name="IC2" library="ElectricNoodleBox" package="DIL16" package3d_urn="urn:adsk.eagle:package:922/2" value="" x="43.18" y="25.4" smashed="yes">
+<attribute name="CATALOGUE" value="3118206" x="43.18" y="25.4" size="1.778" layer="27" display="off"/>
 <attribute name="NAME" x="32.9565" y="24.0665" size="1.27" layer="25" ratio="10" rot="R90"/>
+<attribute name="RETAILER" value="Farnell" x="43.18" y="25.4" size="1.778" layer="27" display="off"/>
 <attribute name="VALUE" x="35.687" y="24.765" size="1.27" layer="27" ratio="10"/>
 </element>
 <element name="IC3" library="ElectricNoodleBox" package="DIL14" package3d_urn="urn:adsk.eagle:package:16407/2" value="" x="21.59" y="25.4" smashed="yes" rot="R180">
+<attribute name="CATALOGUE" value="3005140" x="21.59" y="25.4" size="1.778" layer="27" rot="R180" display="off"/>
 <attribute name="NAME" x="11.176" y="26.8605" size="1.27" layer="25" ratio="10" rot="R270"/>
+<attribute name="RETAILER" value="Farnell" x="21.59" y="25.4" size="1.778" layer="27" rot="R180" display="off"/>
 <attribute name="VALUE" x="28.321" y="26.035" size="1.27" layer="27" ratio="10" rot="R180"/>
 </element>
 <element name="IC4" library="ElectricNoodleBox" package="DIL08" package3d_urn="urn:adsk.eagle:package:29519/2" value="" x="60.96" y="25.4" smashed="yes">
+<attribute name="CATALOGUE" value="1103189" x="60.96" y="25.4" size="1.778" layer="27" display="off"/>
 <attribute name="NAME" x="55.626" y="22.479" size="1.27" layer="25" ratio="10" rot="R90"/>
+<attribute name="RETAILER" value="Farnell" x="60.96" y="25.4" size="1.778" layer="27" display="off"/>
 <attribute name="VALUE" x="57.404" y="24.765" size="1.27" layer="27" ratio="10"/>
 </element>
@@
 <attribute name="VALUE" x="18.415" y="40.3606" size="1.27" layer="27" ratio="10" rot="R270"/>
 </element>
-<element name="R28" library="rcl" library_urn="urn:adsk.eagle:library:334" package="0207/10" package3d_urn="urn:adsk.eagle:package:23491/2" value="2K" x="13.97" y="38.1" smashed="yes" rot="R90">
+<element name="R28" library="rcl" library_urn="urn:adsk.eagle:library:334" package="0207/10" package3d_urn="urn:adsk.eagle:package:23491/2" value="100K" x="13.97" y="38.1" smashed="yes" rot="R90">
 <attribute name="NAME" x="14.6685" y="36.6395" size="1.27" layer="25" ratio="10" rot="R90"/>
 <attribute name="POPULARITY" value="81" x="78.74" y="57.15" size="1.778" layer="27" rot="R90" display="off"/>
@@
 <attribute name="VALUE" x="78.105" y="10.4394" size="1.27" layer="27" ratio="10" rot="R90"/>
 </element>
-<element name="R30" library="rcl" library_urn="urn:adsk.eagle:library:334" package="0207/10" package3d_urn="urn:adsk.eagle:package:23491/2" value="2K" x="26.67" y="38.1" smashed="yes" rot="R270">
+<element name="R30" library="rcl" library_urn="urn:adsk.eagle:library:334" package="0207/10" package3d_urn="urn:adsk.eagle:package:23491/2" value="100K" x="26.67" y="38.1" smashed="yes" rot="R270">
 <attribute name="NAME" x="27.3685" y="36.6395" size="1.27" layer="25" ratio="10" rot="R90"/>
 <attribute name="POPULARITY" value="81" x="-38.1" y="-6.35" size="1.778" layer="27" rot="R270" display="off"/>

Commit message: Fields added and various updates to designs
Parts:
- R1: value 4K7 -> 20K
- R12: value 10K -> 20K
- R16: value 100K -> 47K
Changed lines of the file:
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@@
 <attribute name="VALUE" x="76.2" y="24.765" size="1.27" layer="27" ratio="10" rot="R90"/>
 </element>
-<element name="R1" library="rcl" library_urn="urn:adsk.eagle:library:334" package="0207/10" package3d_urn="urn:adsk.eagle:package:23491/2" value="4K7" x="67.31" y="12.7" smashed="yes" rot="R270">
+<element name="R1" library="rcl" library_urn="urn:adsk.eagle:library:334" package="0207/10" package3d_urn="urn:adsk.eagle:package:23491/2" value="20K" x="67.31" y="12.7" smashed="yes" rot="R270">
 <attribute name="NAME" x="68.0085" y="11.557" size="1.27" layer="25" ratio="10" rot="R90"/>
 <attribute name="POPULARITY" value="81" x="35.56" y="-49.53" size="1.778" layer="27" rot="R270" display="off"/>
@@
 <attribute name="VALUE" x="90.4494" y="32.385" size="1.27" layer="27" ratio="10"/>
 </element>
-<element name="R12" library="rcl" library_urn="urn:adsk.eagle:library:334" package="0207/10" package3d_urn="urn:adsk.eagle:package:23491/2" value="10K" x="67.31" y="38.1" smashed="yes" rot="R270">
+<element name="R12" library="rcl" library_urn="urn:adsk.eagle:library:334" package="0207/10" package3d_urn="urn:adsk.eagle:package:23491/2" value="20K" x="67.31" y="38.1" smashed="yes" rot="R270">
 <attribute name="NAME" x="68.0085" y="36.322" size="1.27" layer="25" ratio="10" rot="R90"/>
 <attribute name="POPULARITY" value="81" x="22.86" y="-31.75" size="1.778" layer="27" rot="R270" display="off"/>
@@
 <attribute name="VALUE" x="83.185" y="35.8394" size="1.27" layer="27" ratio="10" rot="R90"/>
 </element>
-<element name="R16" library="rcl" library_urn="urn:adsk.eagle:library:334" package="0207/10" package3d_urn="urn:adsk.eagle:package:23491/2" value="100K" x="80.01" y="38.1" smashed="yes" rot="R270">
+<element name="R16" library="rcl" library_urn="urn:adsk.eagle:library:334" package="0207/10" package3d_urn="urn:adsk.eagle:package:23491/2" value="47K" x="80.01" y="38.1" smashed="yes" rot="R270">
 <attribute name="NAME" x="80.7085" y="36.322" size="1.27" layer="25" ratio="10" rot="R90"/>
 <attribute name="POPULARITY" value="81" x="30.48" y="-19.05" size="1.778" layer="27" rot="R270" display="off"/>
