File: ModularSeries/PrismTricoreVCO/Panel/PrismNanaPanel.brd (EAGLE design)
At the start: 50.5 x 128.5 mm, 10 parts

Commit message: Fields added and various updates to designs
Routing:
- net S$6: track 27.8 -> 0.00 mm
- net S$5: track 27.8 -> 0.00 mm
- net S$4: track 27.8 -> 0.00 mm
Other:
- board text added: "Track"
- board text removed: "1v/Oct"
Changed lines of the file:
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@@
 <?xml version="1.0" encoding="utf-8"?>
 <!DOCTYPE eagle SYSTEM "eagle.dtd">
-<eagle version="9.6.0">
+<eagle version="9.6.2">
 <drawing>
 <settings>
@@
 </layers>
 <board>
-<fusionsync huburn="a.cGVyc29uYWw6dWUyYjdlNGE0" projecturn="a.cGVyc29uYWw6dWUyYjdlNGE0IzIwMjAwNDA1MjgzMzA0MTgx" f3durn="urn:adsk.wipprod:dm.lineage:JaNhbYIkT3ux4492hbpaaA" pcbguid="9a1187ed-a469-49bd-be31-5f650ae717ec" lastpulledtime="" lastsyncedchangeguid="" latestrevisionid="22984947-b51e-41e3-ae57-f3aa8293c2de" lastsyncedrevisionid="22984947-b51e-41e3-ae57-f3aa8293c2de" lastboardhashguid="f37206f6-6897-1112-536b-1bdd1aae8cd5" lastpushedtime="2020-06-16T15:45:11Z" linktopcb3d="%12"/>
+<fusionsync huburn="a.cGVyc29uYWw6dWUyYjdlNGE0" projecturn="a.cGVyc29uYWw6dWUyYjdlNGE0IzIwMjAwNDA1MjgzMzA0MTgx" f3durn="urn:adsk.wipprod:dm.lineage:JaNhbYIkT3ux4492hbpaaA" pcbguid="9a1187ed-a469-49bd-be31-5f650ae717ec" lastpulledtime="" lastsyncedchangeguid="" latestrevisionid="22984947-b51e-41e3-ae57-f3aa8293c2de" lastsyncedrevisionid="22984947-b51e-41e3-ae57-f3aa8293c2de" lastboardhashguid="f37206f6-6897-1112-536b-1bdd1aae8cd5" lastpushedtime="2020-06-16T15:45:11Z" linktopcb3d="true"/>
 <plain>
 <wire x1="0" y1="-14.25" x2="50.5" y2="-14.25" width="0" layer="20"/>
@@
 <hole x="5.08" y="111.25" drill="3.2"/>
 <hole x="45.72" y="111.25" drill="3.2"/>
-<text x="9.5" y="102" size="1.778" layer="21" font="vector" ratio="12" align="center">1v/Oct</text>
+<text x="9.5" y="102" size="1.778" layer="21" font="vector" ratio="12" align="center">Track</text>
 <text x="9.5" y="82.5" size="1.778" layer="21" font="vector" ratio="12" align="center">FM</text>
 <text x="41" y="102" size="1.778" layer="21" font="vector" ratio="12" align="center">Tri</text>
@@
 <wire x1="41" y1="93.5" x2="30.3" y2="84.6" width="0.1" layer="1" curve="118.016"/>
 </signal>
-<signal name="S$4">
-<wire x1="11.5" y1="23.5" x2="14" y2="19" width="0.5" layer="1"/>
-<wire x1="14" y1="19" x2="11.5" y2="15" width="0.5" layer="1"/>
-<wire x1="11.5" y1="15" x2="9" y2="19" width="0.5" layer="1"/>
-<wire x1="9" y1="19" x2="11.5" y2="23.5" width="0.5" layer="1"/>
-<wire x1="11.5" y1="23.5" x2="12" y2="19" width="0.5" layer="1"/>
-<wire x1="12" y1="19" x2="11.5" y2="15.5" width="0.5" layer="1"/>
-</signal>
-<signal name="S$5">
-<wire x1="4" y1="26" x2="6.5" y2="21.5" width="0.5" layer="1"/>
-<wire x1="6.5" y1="21.5" x2="4" y2="17.5" width="0.5" layer="1"/>
-<wire x1="4" y1="17.5" x2="1.5" y2="21.5" width="0.5" layer="1"/>
-<wire x1="1.5" y1="21.5" x2="4" y2="26" width="0.5" layer="1"/>
-<wire x1="4" y1="26" x2="4.5" y2="21.5" width="0.5" layer="1"/>
-<wire x1="4.5" y1="21.5" x2="4" y2="18" width="0.5" layer="1"/>
-</signal>
-<signal name="S$6">
-<wire x1="19" y1="25.5" x2="21.5" y2="21" width="0.5" layer="1"/>
-<wire x1="21.5" y1="21" x2="19" y2="17" width="0.5" layer="1"/>
-<wire x1="19" y1="17" x2="16.5" y2="21" width="0.5" layer="1"/>
-<wire x1="16.5" y1="21" x2="19" y2="25.5" width="0.5" layer="1"/>
-<wire x1="19" y1="25.5" x2="19.5" y2="21" width="0.5" layer="1"/>
-<wire x1="19.5" y1="21" x2="19" y2="17.5" width="0.5" layer="1"/>
-</signal>
 <signal name="GND">
