File: ModularSeries/FormulaWaveDistortion/FormulaCore.brd (EAGLE design)
At the start: 49.5 x 100 mm, 70 parts, among them Q1 2N3906, Q2 2N3904, Q3 2N3906, Q4 2N3904

Commit message: Formula resistor error corrected in affected files
Parts:
- R18: value 100K -> 10K
Changed lines of the file:
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@@
 </layers>
 <board>
-<fusionsync huburn="a.cGVyc29uYWw6dWUyYjdlNGE0" projecturn="a.cGVyc29uYWw6dWUyYjdlNGE0IzIwMjAwNDA1MjgzMzA0MTgx" f3durn="urn:adsk.wipprod:dm.lineage:mNX1PcfYRniDhO0WAU0ywQ" pcbguid="a3240d91-e514-4e3f-bfbc-c3db2af50738" lastpulledtime="" lastsyncedchangeguid="" latestrevisionid="b2e329d7-1e3c-4786-9d84-b77be482d0da" lastsyncedrevisionid="b2e329d7-1e3c-4786-9d84-b77be482d0da" lastboardhashguid="e19f0be0-f0c6-02eb-c700-d583d042a1fb" lastpushedtime="2020-12-20T16:07:58Z" linktopcb3d="true"/>
+<fusionsync huburn="a.cGVyc29uYWw6dWUyYjdlNGE0" projecturn="a.cGVyc29uYWw6dWUyYjdlNGE0IzIwMjAwNDA1MjgzMzA0MTgx" f3durn="urn:adsk.wipprod:dm.lineage:mNX1PcfYRniDhO0WAU0ywQ" pcbguid="" lastpulledtime="" lastsyncedchangeguid="" latestrevisionid="b2e329d7-1e3c-4786-9d84-b77be482d0da" lastsyncedrevisionid="b2e329d7-1e3c-4786-9d84-b77be482d0da" lastboardhashguid="e19f0be0-f0c6-02eb-c700-d583d042a1fb" lastpushedtime="2020-12-20T16:07:58Z" linktopcb3d="true"/>
 <plain>
 <wire x1="0" y1="95" x2="0" y2="5" width="0" layer="20"/>
@@
 <attribute name="VALUE" x="12.954" y="85.8012" size="1.27" layer="27" ratio="10"/>
 </element>
-<element name="R18" library="rcl" library_urn="urn:adsk.eagle:library:334" package="0207/7" package3d_urn="urn:adsk.eagle:package:23493/2" value="100K" x="15.24" y="71.12" smashed="yes">
+<element name="R18" library="rcl" library_urn="urn:adsk.eagle:library:334" package="0207/7" package3d_urn="urn:adsk.eagle:package:23493/2" value="10K" x="15.24" y="71.12" smashed="yes">
 <attribute name="NAME" x="13.6525" y="70.2945" size="1.27" layer="25" ratio="10"/>
 <attribute name="POPULARITY" value="46" x="53.34" y="15.24" size="1.778" layer="27" display="off"/>
